File: TIVA SMD Header Guide/TIVA SMD Header Guide.kicad_pcb (KiCad board)
At the start: 2 copper layers, 88.9 x 48.3 mm, 1 part

Commit message: Generated Gerbs
Parts:
- added G***: LOGO, MRDT_Silkscreens:MRDT_Logo_4mm, F.Cu at (119.1, 83.7)

Commit message: Created Rev 2
Parts:
- removed the G*** at (119.1, 83.7)
- added G***: LOGO, MRDT_Silkscreens:0_MRDT_Logo_20mm, F.Cu at (121.9, 83.8)
- added G***: LOGO, MRDT_Silkscreens:2_Dahlbot_2.0, B.Cu at (119.4, 83.8)
- added G***: LOGO, MRDT_Silkscreens:2_Nothing_3mm_Cu, F.Cu at (119.4, 83.8)
Other:
- outline, holes or cut-outs redrawn
